Commit message: Fix ros2_control launch race and add SLAM map/config snapshot
Build robot_description directly from the xacro in launch_robot.launch.py
instead of round-tripping through `ros2 param get` against
robot_state_publisher, which raced its node registration on the ROS
graph and made the launch intermittently fail with "Node not found".

Also snapshots the current RViz/Nav2/joystick config tuning and the
SLAM maps produced during real-robot testing (COMEDOR, LIVING_PIEZA,
casa_new, my_map, pieza_new, etc.) that were previously untracked.

Co-Authored-By: Claude Sonnet 5 <noreply@anthropic.com>

File: src/learnbot/description/robot_description.xacro (robot description, xacro)
@@ -43,9 +43,8 @@
     <collision>
       <origin
-        xyz="0 0 0"
-        rpy="0 0 0" />
-      <geometry>
-        <mesh
-          filename="package://learnbot/meshes/base_link.STL" />
+        xyz="0.0001 0 -0.0097"
+        rpy="0 0 0" />
+      <geometry>
+        <box size="0.2086 0.1681 0.0794" />
       </geometry>
     </collision>
@@ -245,6 +244,5 @@
         rpy="0 0 0" />
       <geometry>
-        <mesh
-          filename="package://learnbot/meshes/caster_wheel_link.STL" />
+        <sphere radius="0.016" />
       </geometry>
     </collision>
@@ -349,8 +347,7 @@
       <origin
         xyz="0 0 0"
-        rpy="0 0 0" />
-      <geometry>
-        <mesh
-          filename="package://learnbot/meshes/right_wheel_link.STL" />
+        rpy="1.5707963267948966 0 0" />
+      <geometry>
+        <cylinder radius="0.033" length="0.032" />
       </geometry>
     </collision>
@@ -461,8 +458,7 @@
       <origin
         xyz="0 0 0"
-        rpy="0 0 0" />
-      <geometry>
-        <mesh
-          filename="package://learnbot/meshes/left_wheel_link.STL" />
+        rpy="1.5707963267948966 0 0" />
+      <geometry>
+        <cylinder radius="0.033" length="0.032" />
       </geometry>
     </collision>

File: src/learnbot/description/robot_gazebo.xacro (robot description, xacro)
@@ -37,5 +37,5 @@
     <sensor type="ray" name="lidar">
       <pose>0 0 0 0 0 0</pose>
-      <visualize>false</visualize>
+      <visualize>true</visualize>
       <update_rate>10</update_rate>
       <ray>
